File: KiCad/40Hz_S2/40Hz_S2.kicad_pcb (KiCad board)
At the start: 2 copper layers, 59.2 x 43.8 mm, 15 parts, among them J1 PWR, J2 Audio, J3 LED, Q1 IRF540N, U1 WeMos_S2_mini

Commit message: updated grp files
Parts:
- Q1: value IRF540N -> CSD19531KCS
Routing:
- net GND: track 178.4 -> 191.5 mm
- net Audio: track 11.9 -> 11.8 mm, vias 1 -> 0
- net (no net): vias 3 -> 4
Other:
- board text added: "4Ω or 8Ω"
- board text added: "Add S2 headers first before attaching display"
- board text added: "For DAC output, set to 0k."
- board text added: "Set 50k trim to center"
- board text added: "Ver. 0.3"
- board text added: "What we think, we become."
- board text added: "to keep output below +0.6V."
- board text removed: "(4Ω)"
- board text removed: "(5VDC)"
