File: KiCad/40Hz_S2/40Hz_S2.kicad_sch (KiCad schematic)
At the start: 15 parts, among them J1 PWR, J2 Audio, J3 LED, Q1 CSD19531KCS, U1 WeMos_S2_mini

Commit message: updated grp files
Parts:
- U1: footprint Module:WEMOS_S2_mini -> SamacSys_Parts:WEMOS_S2_mini_no_inner_row
Changed lines of the file:
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@@
 			)
 		)
-		(property "Footprint" "Module:WEMOS_S2_mini"
+		(property "Footprint" "SamacSys_Parts:WEMOS_S2_mini_no_inner_row"
 			(at 186.69 157.48 0)
 			(effects
